File: Kicad Files/i2c_multiplexers.kicad_sch (KiCad schematic)
At the start: 9 parts, among them U3 PCA9548APW

Commit message: Various updates and fixes
Parts:
- U3: footprint SFLibrary:SOP65P640X120-24N -> PCA9548APW:SOP65P640X120-24N; symbol SFLibrary:PCA9548APW -> SF Library:PCA9548APW
Changed lines of the file:
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@@
 (kicad_sch
-	(version 20231120)
+	(version 20250114)
 	(generator "eeschema")
-	(generator_version "8.0")
+	(generator_version "9.0")
 	(paper "A4")
 	(junction
@@
 	)
 	(symbol
-		(lib_id "SFLibrary:PCA9548APW")
+		(lib_id "SF Library:PCA9548APW")
 		(at 124.46 88.9 0)
 		(unit 1)
@@
 			)
 		)
-		(property "Footprint" "SFLibrary:SOP65P640X120-24N"
+		(property "Footprint" "PCA9548APW:SOP65P640X120-24N"
 			(at 124.46 88.9 0)
 			(effects
