File: Kicad Files/powerconn.kicad_sch (KiCad schematic)
At the start: 19 parts, among them J3 BootLoader, J4 PJ-102A, P1 USB_C_Plug_USB2.0, U4 AMS1117-3.3, U5 CH340G, U6 AMS1117-5.0

Commit message: Various updates and fixes
Changed lines of the file:
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@@
 (kicad_sch
-	(version 20231120)
+	(version 20250114)
 	(generator "eeschema")
-	(generator_version "8.0")
+	(generator_version "9.0")
 	(paper "A4")
 	(junction
