File: 7Segments/7segments.kicad_pcb (KiCad board)
At the start: 2 copper layers, 51 x 20 mm, 11 parts, among them J1 KHZ_UP, J2 KHZ_DOWN, J3 MHZ_UP, J4 MHZ_DOWN, J5 Conn_02x08_Top_Bottom_Shielded

Commit message: Clear the ERC errors and the real DRC findings on all four boards
7Segments
- J5 used Conn_02x08_Top_Bottom_Shielded on an IDC header with no shield
  pad: ERC flagged the SH pin, DRC a net conflict. It is now the plain
  Conn_02x08_Top_Bottom, like J7/J8 on the MainPanel; pins 1-16 sit at
  the same points, so nothing else moved.
- GND had no driver: PWR_FLAG added.

BoardPanel
- P1 read "USB_C_Plug_USB2.0" on a USB-B connector: value now USB_B.
- +5V had no driver: pin 3 (+VOUT) of the P78A05 symbol is now a power
  output, in the schematic and in Libraries/RMP.kicad_sym. A PWR_FLAG
  there would clash with the pin.

MainPanel
- A stray no-connect flag and a second PWR_FLAG on the same net removed.

LedsPanel
- Q1 (IRLZ44N) pins were "unspecified": now passive, as in the overhead
  panel's library.
- Q1 courtyard: the two zero-length segments are gone, in the library
  footprint and on the board. The rest was already a closed outline
  around all three pads.
- J1 value on the board brought in line with the schematic (From_Main).

ERC is now 0 on 7Segments, LedsPanel and MainPanel. BoardPanel keeps one
warning, P1's USB_B symbol differing from the KiCad 10 library; that and
the DRC library/field mismatches go with Update Symbols/Footprints from
Library, as on the FCU. Netlists are unchanged apart from J5's SH node
and P1's value. Copper plots to the same geometry.

Co-Authored-By: Claude Opus 5.5 <noreply@anthropic.com>
Parts:
- J5: value Conn_02x08_Top_Bottom_Shielded -> Conn_02x08_Top_Bottom
Changed lines of the file:
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@@
 			)
 		)
-		(property "Value" "Conn_02x08_Top_Bottom_Shielded"
+		(property "Value" "Conn_02x08_Top_Bottom"
 			(at 1.27 -23.88 90)
 			(layer "B.Fab")
