File: MainPanel/MainPanel.kicad_sch (KiCad schematic)
At the start: 24 parts, among them J1 To_Led, J2 LED_From_Board, J3 Main_From_Board, J4 Power Switch, J5 Rotary KHz, J6 Rotary MHz

Commit message: Bring the custom parts into Libraries/, shared by all four boards
Six parts came from libraries that live only on the author's PC (SF
Library, IRLZ44N, P78A05-1000, Custom_Footprints, PCM_SFLibrary and the
Digi-Key PCM libraries). Their 3D models pointed at a KiCad 9 3rdparty
folder that no longer exists, so the boards rendered without them.

They now sit in Libraries/ under one nickname, RMP, as the overhead
panel does with OVHD:

  RMP.kicad_sym   MAX7219CWGT, IRLZ44NSTRLPBF, P78A05-1000, PJ-102A,
                  1825910-6, MJTP1230, taken from the schematic caches,
                  i.e. the symbols the boards were drawn with
  RMP.pretty      CONV_P78A05-1000, SOIC127P1032X265-24N,
                  TQFP100-0.5-14X14MM, NMOSGDS_D2PAK_INF, the PJ-102A
                  barrel jack and the MJTP1230 switch, copied from the
                  personal libraries (DRC found no difference from the
                  placed copies), with the 3D model of each board
                  instance added where the library had none
  3dmodels/       the seven vendor STEP files the boards use

Each board has a project sym-lib-table and fp-lib-table pointing at
${KIPRJMOD}/../Libraries, and every custom model path is now
${KIPRJMOD}/../Libraries/3dmodels/..., which resolves on any machine.

Netlists are unchanged apart from the library nickname in the footprint
field of U1, U2, S1, J1 (BoardPanel), Q1 (LedsPanel), U1, U2 and S1-S13
(MainPanel). Copper plots to the same geometry. ERC drops the missing-
library warnings: BoardPanel 4 -> 2, MainPanel 17 -> 2.

DRC no longer lists the malformed courtyard of the LedsPanel Q1, but its
courtyard still holds zero-length segments: it is fixed separately.

Co-Authored-By: Claude Opus 5.5 <noreply@anthropic.com>
Parts:
- S1, S10, S11, S12, S13, S2, S3, S4, S5, S6, S7, S8, S9: footprint digikey-footprints:Switch_Tactile_THT_6x6mm_MJTP1230 -> RMP:Switch_Tactile_THT_6x6mm_MJTP1230; symbol PCM_dk_Tactile-Switches:MJTP1230 -> RMP:MJTP1230
Changed lines of the file:
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@@
 	)
 	(symbol
-		(lib_id "PCM_dk_Tactile-Switches:MJTP1230")
+		(lib_id "RMP:MJTP1230")
 		(at 105.41 91.44 0)
 		(unit 1)
@@
 			)
 		)
-		(property "Footprint" "digikey-footprints:Switch_Tactile_THT_6x6mm_MJTP1230"
+		(property "Footprint" "RMP:Switch_Tactile_THT_6x6mm_MJTP1230"
 			(at 110.49 86.36 0)
 			(hide yes)
@@
 	)
 	(symbol
-		(lib_id "PCM_dk_Tactile-Switches:MJTP1230")
+		(lib_id "RMP:MJTP1230")
 		(at 105.41 50.8 0)
 		(unit 1)
@@
 			)
 		)
-		(property "Footprint" "digikey-footprints:Switch_Tactile_THT_6x6mm_MJTP1230"
+		(property "Footprint" "RMP:Switch_Tactile_THT_6x6mm_MJTP1230"
 			(at 110.49 45.72 0)
 			(hide yes)
@@
 	)
 	(symbol
-		(lib_id "PCM_dk_Tactile-Switches:MJTP1230")
+		(lib_id "RMP:MJTP1230")
 		(at 76.2 90.17 0)
 		(unit 1)
@@
 			)
 		)
-		(property "Footprint" "digikey-footprints:Switch_Tactile_THT_6x6mm_MJTP1230"
+		(property "Footprint" "RMP:Switch_Tactile_THT_6x6mm_MJTP1230"
 			(at 81.28 85.09 0)
 			(hide yes)
@@
 	)
 	(symbol
-		(lib_id "PCM_dk_Tactile-Switches:MJTP1230")
+		(lib_id "RMP:MJTP1230")
 		(at 105.41 107.95 0)
 		(unit 1)
@@
 			)
 		)
-		(property "Footprint" "digikey-footprints:Switch_Tactile_THT_6x6mm_MJTP1230"
+		(property "Footprint" "RMP:Switch_Tactile_THT_6x6mm_MJTP1230"
 			(at 110.49 102.87 0)
 			(hide yes)
@@
 	)
 	(symbol
-		(lib_id "PCM_dk_Tactile-Switches:MJTP1230")
+		(lib_id "RMP:MJTP1230")
 		(at 46.99 50.8 0)
 		(unit 1)
@@
 			)
 		)
-		(property "Footprint" "digikey-footprints:Switch_Tactile_THT_6x6mm_MJTP1230"
+		(property "Footprint" "RMP:Switch_Tactile_THT_6x6mm_MJTP1230"
 			(at 52.07 45.72 0)
 			(hide yes)
@@
 	)
 	(symbol
-		(lib_id "PCM_dk_Tactile-Switches:MJTP1230")
+		(lib_id "RMP:MJTP1230")
 		(at 105.41 72.39 0)
 		(unit 1)
@@
 			)
 		)
-		(property "Footprint" "digikey-footprints:Switch_Tactile_THT_6x6mm_MJTP1230"
+		(property "Footprint" "RMP:Switch_Tactile_THT_6x6mm_MJTP1230"
 			(at 110.49 67.31 0)
 			(hide yes)
@@
 	)
 	(symbol
-		(lib_id "PCM_dk_Tactile-Switches:MJTP1230")
+		(lib_id "RMP:MJTP1230")
 		(at 129.54 30.48 0)
 		(unit 1)
@@
 			)
 		)
-		(property "Footprint" "digikey-footprints:Switch_Tactile_THT_6x6mm_MJTP1230"
+		(property "Footprint" "RMP:Switch_Tactile_THT_6x6mm_MJTP1230"
 			(at 134.62 25.4 0)
 			(hide yes)
@@
 	)
 	(symbol
-		(lib_id "PCM_dk_Tactile-Switches:MJTP1230")
+		(lib_id "RMP:MJTP1230")
 		(at 46.99 72.39 0)
 		(unit 1)
@@
 			)
 		)
-		(property "Footprint" "digikey-footprints:Switch_Tactile_THT_6x6mm_MJTP1230"
+		(property "Footprint" "RMP:Switch_Tactile_THT_6x6mm_MJTP1230"
 			(at 52.07 67.31 0)
 			(hide yes)
@@
 	)
 	(symbol
-		(lib_id "PCM_dk_Tactile-Switches:MJTP1230")
+		(lib_id "RMP:MJTP1230")
 		(at 76.2 72.39 0)
 		(unit 1)
@@
 			)
 		)
-		(property "Footprint" "digikey-footprints:Switch_Tactile_THT_6x6mm_MJTP1230"
+		(property "Footprint" "RMP:Switch_Tactile_THT_6x6mm_MJTP1230"
 			(at 81.28 67.31 0)
 			(hide yes)
@@
 	)
 	(symbol
-		(lib_id "PCM_dk_Tactile-Switches:MJTP1230")
+		(lib_id "RMP:MJTP1230")
 		(at 46.99 90.17 0)
 		(unit 1)
@@
 			)
 		)
-		(property "Footprint" "digikey-footprints:Switch_Tactile_THT_6x6mm_MJTP1230"
+		(property "Footprint" "RMP:Switch_Tactile_THT_6x6mm_MJTP1230"
 			(at 52.07 85.09 0)
 			(hide yes)
@@
 	)
 	(symbol
-		(lib_id "PCM_dk_Tactile-Switches:MJTP1230")
+		(lib_id "RMP:MJTP1230")
 		(at 76.2 107.95 0)
 		(unit 1)
@@
 			)
 		)
-		(property "Footprint" "digikey-footprints:Switch_Tactile_THT_6x6mm_MJTP1230"
+		(property "Footprint" "RMP:Switch_Tactile_THT_6x6mm_MJTP1230"
 			(at 81.28 102.87 0)
 			(hide yes)
@@
 	)
 	(symbol
-		(lib_id "PCM_dk_Tactile-Switches:MJTP1230")
+		(lib_id "RMP:MJTP1230")
 		(at 46.99 107.95 0)
 		(unit 1)
@@
 			)
 		)
-		(property "Footprint" "digikey-footprints:Switch_Tactile_THT_6x6mm_MJTP1230"
+		(property "Footprint" "RMP:Switch_Tactile_THT_6x6mm_MJTP1230"
 			(at 52.07 102.87 0)
 			(hide yes)
@@
 	)
 	(symbol
-		(lib_id "PCM_dk_Tactile-Switches:MJTP1230")
+		(lib_id "RMP:MJTP1230")
 		(at 76.2 50.8 0)
 		(unit 1)
@@
 			)
 		)
-		(property "Footprint" "digikey-footprints:Switch_Tactile_THT_6x6mm_MJTP1230"
+		(property "Footprint" "RMP:Switch_Tactile_THT_6x6mm_MJTP1230"
 			(at 81.28 45.72 0)
 			(hide yes)

Commit message: Clear the ERC errors and the real DRC findings on all four boards
7Segments
- J5 used Conn_02x08_Top_Bottom_Shielded on an IDC header with no shield
  pad: ERC flagged the SH pin, DRC a net conflict. It is now the plain
  Conn_02x08_Top_Bottom, like J7/J8 on the MainPanel; pins 1-16 sit at
  the same points, so nothing else moved.
- GND had no driver: PWR_FLAG added.

BoardPanel
- P1 read "USB_C_Plug_USB2.0" on a USB-B connector: value now USB_B.
- +5V had no driver: pin 3 (+VOUT) of the P78A05 symbol is now a power
  output, in the schematic and in Libraries/RMP.kicad_sym. A PWR_FLAG
  there would clash with the pin.

MainPanel
- A stray no-connect flag and a second PWR_FLAG on the same net removed.

LedsPanel
- Q1 (IRLZ44N) pins were "unspecified": now passive, as in the overhead
  panel's library.
- Q1 courtyard: the two zero-length segments are gone, in the library
  footprint and on the board. The rest was already a closed outline
  around all three pads.
- J1 value on the board brought in line with the schematic (From_Main).

ERC is now 0 on 7Segments, LedsPanel and MainPanel. BoardPanel keeps one
warning, P1's USB_B symbol differing from the KiCad 10 library; that and
the DRC library/field mismatches go with Update Symbols/Footprints from
Library, as on the FCU. Netlists are unchanged apart from J5's SH node
and P1's value. Copper plots to the same geometry.

Co-Authored-By: Claude Opus 5.5 <noreply@anthropic.com>
Connections:
- no-connect marks 17 -> 16
Changed lines of the file:
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@@
-	)
-	(no_connect
-		(at 259.08 160.02)
 	)
 	(no_connect
