File: MainPanel/max7219.kicad_sch (KiCad schematic)
At the start: 11 parts, among them J7 ACTIVE_DISPLAY, J8 STBY_DISPLAY, J9 DisplayFromBoard, U1 ACTIVE DISPLAY, U2 STANDBY DISPLAY

Commit message: Bring the custom parts into Libraries/, shared by all four boards
Six parts came from libraries that live only on the author's PC (SF
Library, IRLZ44N, P78A05-1000, Custom_Footprints, PCM_SFLibrary and the
Digi-Key PCM libraries). Their 3D models pointed at a KiCad 9 3rdparty
folder that no longer exists, so the boards rendered without them.

They now sit in Libraries/ under one nickname, RMP, as the overhead
panel does with OVHD:

  RMP.kicad_sym   MAX7219CWGT, IRLZ44NSTRLPBF, P78A05-1000, PJ-102A,
                  1825910-6, MJTP1230, taken from the schematic caches,
                  i.e. the symbols the boards were drawn with
  RMP.pretty      CONV_P78A05-1000, SOIC127P1032X265-24N,
                  TQFP100-0.5-14X14MM, NMOSGDS_D2PAK_INF, the PJ-102A
                  barrel jack and the MJTP1230 switch, copied from the
                  personal libraries (DRC found no difference from the
                  placed copies), with the 3D model of each board
                  instance added where the library had none
  3dmodels/       the seven vendor STEP files the boards use

Each board has a project sym-lib-table and fp-lib-table pointing at
${KIPRJMOD}/../Libraries, and every custom model path is now
${KIPRJMOD}/../Libraries/3dmodels/..., which resolves on any machine.

Netlists are unchanged apart from the library nickname in the footprint
field of U1, U2, S1, J1 (BoardPanel), Q1 (LedsPanel), U1, U2 and S1-S13
(MainPanel). Copper plots to the same geometry. ERC drops the missing-
library warnings: BoardPanel 4 -> 2, MainPanel 17 -> 2.

DRC no longer lists the malformed courtyard of the LedsPanel Q1, but its
courtyard still holds zero-length segments: it is fixed separately.

Co-Authored-By: Claude Opus 5.5 <noreply@anthropic.com>
Parts:
- U1, U2: footprint Custom_Footprints:SOIC127P1032X265-24N -> RMP:SOIC127P1032X265-24N; symbol SF Library:MAX7219CWGT -> RMP:MAX7219CWGT
Changed lines of the file:
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@@
 	)
 	(symbol
-		(lib_id "SF Library:MAX7219CWGT")
+		(lib_id "RMP:MAX7219CWGT")
 		(at 105.41 66.04 0)
 		(unit 1)
@@
 			)
 		)
-		(property "Footprint" "Custom_Footprints:SOIC127P1032X265-24N"
+		(property "Footprint" "RMP:SOIC127P1032X265-24N"
 			(at 105.41 66.04 0)
 			(hide yes)
@@
 	)
 	(symbol
-		(lib_id "SF Library:MAX7219CWGT")
+		(lib_id "RMP:MAX7219CWGT")
 		(at 228.6 77.47 0)
 		(unit 1)
@@
 			)
 		)
-		(property "Footprint" "Custom_Footprints:SOIC127P1032X265-24N"
+		(property "Footprint" "RMP:SOIC127P1032X265-24N"
 			(at 228.6 77.47 0)
 			(hide yes)

Commit message: Chain the two MAX7219 on the MainPanel, as the built unit is wired
The schematic had both drivers on the MCU's DIN with a LOAD each (D67 for
the Active, D68 for the Standby) and both DOUT unconnected. The board in
use only works because two wires were added by hand: LOAD to LOAD, and
the Standby's DOUT to the Active's DIN. MobiFlight drives it as one LED
module of two devices on CS D68: connector 1 is the Standby, the first
in the chain, connector 2 the Active.

The design now matches:

  DIN         J9 pin 5 (D23) -> U2 (Standby) pin 1 only
  ACTIVE_DIN  U2 pin 24 (DOUT) -> U1 (Active) pin 1
  LOAD        J9 pin 6 (D68) -> U1 and U2 pin 12
  J9 pin 3    (D67) no longer used, flagged no-connect

The BoardPanel and the board config do not change. The old DIN branch
to U1 and the ACTIVE_LOAD track were removed; the two new connections
were routed interactively in KiCad (VHF2_BTN was shoved), then the GND
zones refilled. DRC: 0 unconnected, no clearance violation; the 15
remaining entries are the same library and field warnings as before.
Schematic parity unchanged.

On a board built from the old files, an Active display that shows the
odd wrong segment points at U1 pin 1: it is still tied to D23 by copper,
and with the hand wire it has two drivers.

Co-Authored-By: Claude Opus 5.5 <noreply@anthropic.com>
Connections:
- net DIN: no longer U1.1 (DIN)
- net ACTIVE_DIN: now reaches U2.24 (DOUT)
- net ACTIVE_DIN: now also U1.1 (DIN)
- net ACTIVE_LOAD: no longer names the net of J9.3 (Pin_3)
- net ACTIVE_LOAD: no longer U1.12 (LOAD)
- net STBY_LOAD renamed LOAD
- net LOAD: now also U1.12 (LOAD)
Changed lines of the file:
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@@
 		(at 123.19 50.8)
 	)
-	(no_connect
-		(at 246.38 44.45)
+	(label "ACTIVE_DIN"
+		(at 246.38 44.45 0)
+		(effects
+			(font
+				(size 1.27 1.27)
+			)
+			(justify left bottom)
+		)
 	)
 	(no_connect
@@
 		)
 	)
-	(label "DIN"
+	(label "ACTIVE_DIN"
 		(at 87.63 35.56 180)
 		(effects
@@
 		)
 	)
-	(label "STBY_LOAD"
+	(label "LOAD"
 		(at 210.82 49.53 180)
 		(effects
@@
 		)
 	)
-	(label "ACTIVE_LOAD"
-		(at 52.07 171.45 180)
-		(effects
-			(font
-				(size 1.27 1.27)
-			)
-			(justify right bottom)
-		)
+	(no_connect
+		(at 52.07 171.45)
 	)
 	(label "DIN"
@@
 		)
 	)
-	(label "STBY_LOAD"
+	(label "LOAD"
 		(at 64.77 171.45 0)
 		(effects
@@
 		)
 	)
-	(label "ACTIVE_LOAD"
+	(label "LOAD"
 		(at 87.63 38.1 180)
 		(effects

Commit message: Clear the ERC errors and the real DRC findings on all four boards
7Segments
- J5 used Conn_02x08_Top_Bottom_Shielded on an IDC header with no shield
  pad: ERC flagged the SH pin, DRC a net conflict. It is now the plain
  Conn_02x08_Top_Bottom, like J7/J8 on the MainPanel; pins 1-16 sit at
  the same points, so nothing else moved.
- GND had no driver: PWR_FLAG added.

BoardPanel
- P1 read "USB_C_Plug_USB2.0" on a USB-B connector: value now USB_B.
- +5V had no driver: pin 3 (+VOUT) of the P78A05 symbol is now a power
  output, in the schematic and in Libraries/RMP.kicad_sym. A PWR_FLAG
  there would clash with the pin.

MainPanel
- A stray no-connect flag and a second PWR_FLAG on the same net removed.

LedsPanel
- Q1 (IRLZ44N) pins were "unspecified": now passive, as in the overhead
  panel's library.
- Q1 courtyard: the two zero-length segments are gone, in the library
  footprint and on the board. The rest was already a closed outline
  around all three pads.
- J1 value on the board brought in line with the schematic (From_Main).

ERC is now 0 on 7Segments, LedsPanel and MainPanel. BoardPanel keeps one
warning, P1's USB_B symbol differing from the KiCad 10 library; that and
the DRC library/field mismatches go with Update Symbols/Footprints from
Library, as on the FCU. Netlists are unchanged apart from J5's SH node
and P1's value. Copper plots to the same geometry.

Co-Authored-By: Claude Opus 5.5 <noreply@anthropic.com>
Changed lines of the file:
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@@
-	)
-	(symbol
-		(lib_id "power:PWR_FLAG")
-		(at 29.21 168.91 180)
-		(unit 1)
-		(body_style 1)
-		(exclude_from_sim no)
-		(in_bom yes)
-		(on_board yes)
-		(in_pos_files yes)
-		(dnp no)
-		(fields_autoplaced yes)
-		(property "Reference" "#FLG02"
-			(at 29.21 170.815 0)
-			(hide yes)
-			(show_name no)
-			(do_not_autoplace no)
-			(effects
-				(font
-					(size 1.27 1.27)
-				)
-			)
-		)
-		(property "Value" "PWR_FLAG"
-			(at 29.21 173.99 0)
-			(show_name no)
-			(do_not_autoplace no)
-			(effects
-				(font
-					(size 1.27 1.27)
-				)
-			)
-		)
-		(property "Footprint" ""
-			(at 29.21 168.91 0)
-			(hide yes)
-			(show_name no)
-			(do_not_autoplace no)
-			(effects
-				(font
-					(size 1.27 1.27)
-				)
-			)
-		)
-		(property "Datasheet" ""
-			(at 29.21 168.91 0)
-			(hide yes)
-			(show_name no)
-			(do_not_autoplace no)
-			(effects
-				(font
-					(size 1.27 1.27)
-				)
-			)
-		)
-		(property "Description" "Special symbol for telling ERC where power comes from"
-			(at 29.21 168.91 0)
-			(hide yes)
-			(show_name no)
-			(do_not_autoplace no)
-			(effects
-				(font
-					(size 1.27 1.27)
-				)
-			)
-		)
-		(pin "1"
-		)
-		(instances
-			(project "MainPanel"
-				(path "/eb52c842-e2cb-42c4-b3df-d076726fc248/d5878c5f-367a-496b-83f6-db933576c882"
-					(reference "#FLG02")
-					(unit 1)
-				)
-			)
-		)
 	)
 	(symbol
