File: MainPanel/MainPanel.kicad_pcb (KiCad board)
At the start: 2 copper layers, 122 x 79.9 mm, 35 parts, among them J1 To_Led, J2 LED_From_Board, J3 Main_From_Board, J4 Power Switch, J5 Rotary KHz, J6 Rotary MHz, J7 ACTIVE_DISPLAY, J8 STBY_DISPLAY, J9 DisplayFromBoard, U1 ACTIVE DISPLAY, U2 STANDBY DISPLAY

Commit message: Bring the custom parts into Libraries/, shared by all four boards
Six parts came from libraries that live only on the author's PC (SF
Library, IRLZ44N, P78A05-1000, Custom_Footprints, PCM_SFLibrary and the
Digi-Key PCM libraries). Their 3D models pointed at a KiCad 9 3rdparty
folder that no longer exists, so the boards rendered without them.

They now sit in Libraries/ under one nickname, RMP, as the overhead
panel does with OVHD:

  RMP.kicad_sym   MAX7219CWGT, IRLZ44NSTRLPBF, P78A05-1000, PJ-102A,
                  1825910-6, MJTP1230, taken from the schematic caches,
                  i.e. the symbols the boards were drawn with
  RMP.pretty      CONV_P78A05-1000, SOIC127P1032X265-24N,
                  TQFP100-0.5-14X14MM, NMOSGDS_D2PAK_INF, the PJ-102A
                  barrel jack and the MJTP1230 switch, copied from the
                  personal libraries (DRC found no difference from the
                  placed copies), with the 3D model of each board
                  instance added where the library had none
  3dmodels/       the seven vendor STEP files the boards use

Each board has a project sym-lib-table and fp-lib-table pointing at
${KIPRJMOD}/../Libraries, and every custom model path is now
${KIPRJMOD}/../Libraries/3dmodels/..., which resolves on any machine.

Netlists are unchanged apart from the library nickname in the footprint
field of U1, U2, S1, J1 (BoardPanel), Q1 (LedsPanel), U1, U2 and S1-S13
(MainPanel). Copper plots to the same geometry. ERC drops the missing-
library warnings: BoardPanel 4 -> 2, MainPanel 17 -> 2.

DRC no longer lists the malformed courtyard of the LedsPanel Q1, but its
courtyard still holds zero-length segments: it is fixed separately.

Co-Authored-By: Claude Opus 5.5 <noreply@anthropic.com>
Parts:
- S1, S10, S11, S12, S13, S2, S3, S4, S5, S6, S7, S8, S9: footprint digikey-footprints:Switch_Tactile_THT_6x6mm_MJTP1230 -> RMP:Switch_Tactile_THT_6x6mm_MJTP1230
- U1, U2: footprint Custom_Footprints:SOIC127P1032X265-24N -> RMP:SOIC127P1032X265-24N
Changed lines of the file:
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@@
 		)
 	)
-	(footprint "digikey-footprints:Switch_Tactile_THT_6x6mm_MJTP1230"
+	(footprint "RMP:Switch_Tactile_THT_6x6mm_MJTP1230"
 		(layer "F.Cu")
 		(at 44.925 64.4)
@@
 		)
 		(embedded_fonts no)
-		(model "${KICAD9_3RD_PARTY}/3dmodels/1825910-6.STEP"
+		(model "${KIPRJMOD}/../Libraries/3dmodels/1825910-6.STEP"
 			(offset
 				(xyz 3.2 -2.2 0)
@@
 		)
 	)
-	(footprint "digikey-footprints:Switch_Tactile_THT_6x6mm_MJTP1230"
+	(footprint "RMP:Switch_Tactile_THT_6x6mm_MJTP1230"
 		(layer "F.Cu")
 		(at 27.925 79.4)
@@
 		)
 		(embedded_fonts no)
-		(model "${KICAD9_3RD_PARTY}/3dmodels/1825910-6.STEP"
+		(model "${KIPRJMOD}/../Libraries/3dmodels/1825910-6.STEP"
 			(offset
 				(xyz 3.2 -2.2 0)
@@
 		)
 	)
-	(footprint "digikey-footprints:Switch_Tactile_THT_6x6mm_MJTP1230"
+	(footprint "RMP:Switch_Tactile_THT_6x6mm_MJTP1230"
 		(layer "F.Cu")
 		(at 27.925 99.9)
@@
 		)
 		(embedded_fonts no)
-		(model "${KICAD9_3RD_PARTY}/3dmodels/1825910-6.STEP"
+		(model "${KIPRJMOD}/../Libraries/3dmodels/1825910-6.STEP"
 			(offset
 				(xyz 3.2 -2.2 0)
@@
 		)
 	)
-	(footprint "digikey-footprints:Switch_Tactile_THT_6x6mm_MJTP1230"
+	(footprint "RMP:Switch_Tactile_THT_6x6mm_MJTP1230"
 		(layer "F.Cu")
 		(at 61.925 99.9)
@@
 		)
 		(embedded_fonts no)
-		(model "${KICAD9_3RD_PARTY}/3dmodels/1825910-6.STEP"
+		(model "${KIPRJMOD}/../Libraries/3dmodels/1825910-6.STEP"
 			(offset
 				(xyz 3.2 -2.2 0)
@@
 		)
 	)
-	(footprint "digikey-footprints:Switch_Tactile_THT_6x6mm_MJTP1230"
+	(footprint "RMP:Switch_Tactile_THT_6x6mm_MJTP1230"
 		(layer "F.Cu")
 		(at 112.925 99.9)
@@
 		)
 		(embedded_fonts no)
-		(model "${KICAD9_3RD_PARTY}/3dmodels/1825910-6.STEP"
+		(model "${KIPRJMOD}/../Libraries/3dmodels/1825910-6.STEP"
 			(offset
 				(xyz 3.2 -2.2 0)
@@
 		)
 	)
-	(footprint "digikey-footprints:Switch_Tactile_THT_6x6mm_MJTP1230"
+	(footprint "RMP:Switch_Tactile_THT_6x6mm_MJTP1230"
 		(layer "F.Cu")
 		(at 61.925 79.4)
@@
 		)
 		(embedded_fonts no)
-		(model "${KICAD9_3RD_PARTY}/3dmodels/1825910-6.STEP"
+		(model "${KIPRJMOD}/../Libraries/3dmodels/1825910-6.STEP"
 			(offset
 				(xyz 3.2 -2.2 0)
@@
 		)
 	)
-	(footprint "digikey-footprints:Switch_Tactile_THT_6x6mm_MJTP1230"
+	(footprint "RMP:Switch_Tactile_THT_6x6mm_MJTP1230"
 		(layer "F.Cu")
 		(at 27.925 64.4)
@@
 		)
 		(embedded_fonts no)
-		(model "${KICAD9_3RD_PARTY}/3dmodels/1825910-6.STEP"
+		(model "${KIPRJMOD}/../Libraries/3dmodels/1825910-6.STEP"
 			(offset
 				(xyz 3.2 -2.2 0)
@@
 		)
 	)
-	(footprint "digikey-footprints:Switch_Tactile_THT_6x6mm_MJTP1230"
+	(footprint "RMP:Switch_Tactile_THT_6x6mm_MJTP1230"
 		(layer "F.Cu")
 		(at 44.925 99.9)
@@
 		)
 		(embedded_fonts no)
-		(model "${KICAD9_3RD_PARTY}/3dmodels/1825910-6.STEP"
+		(model "${KIPRJMOD}/../Libraries/3dmodels/1825910-6.STEP"
 			(offset
 				(xyz 3.2 -2.2 0)
@@
 		(embedded_fonts no)
 	)
-	(footprint "digikey-footprints:Switch_Tactile_THT_6x6mm_MJTP1230"
+	(footprint "RMP:Switch_Tactile_THT_6x6mm_MJTP1230"
 		(layer "F.Cu")
 		(at 61.925 64.4)
@@
 		)
 		(embedded_fonts no)
-		(model "${KICAD9_3RD_PARTY}/3dmodels/1825910-6.STEP"
+		(model "${KIPRJMOD}/../Libraries/3dmodels/1825910-6.STEP"
 			(offset
 				(xyz 3.2 -2.2 0)
@@
 		(embedded_fonts no)
 	)
-	(footprint "digikey-footprints:Switch_Tactile_THT_6x6mm_MJTP1230"
+	(footprint "RMP:Switch_Tactile_THT_6x6mm_MJTP1230"
 		(layer "F.Cu")
 		(at 95.925 99.9)
@@
 		)
 		(embedded_fonts no)
-		(model "${KICAD9_3RD_PARTY}/3dmodels/1825910-6.STEP"
+		(model "${KIPRJMOD}/../Libraries/3dmodels/1825910-6.STEP"
 			(offset
 				(xyz 3.2 -2.2 0)
@@
 		)
 	)
-	(footprint "digikey-footprints:Switch_Tactile_THT_6x6mm_MJTP1230"
+	(footprint "RMP:Switch_Tactile_THT_6x6mm_MJTP1230"
 		(layer "F.Cu")
 		(at 78.925 79.4)
@@
 		)
 		(embedded_fonts no)
-		(model "${KICAD9_3RD_PARTY}/3dmodels/1825910-6.STEP"
+		(model "${KIPRJMOD}/../Libraries/3dmodels/1825910-6.STEP"
 			(offset
 				(xyz 3.2 -2.2 0)
@@
 		)
 	)
-	(footprint "digikey-footprints:Switch_Tactile_THT_6x6mm_MJTP1230"
+	(footprint "RMP:Switch_Tactile_THT_6x6mm_MJTP1230"
 		(layer "F.Cu")
 		(at 79.925 42.4)
@@
 		)
 		(embedded_fonts no)
-		(model "${KICAD9_3RD_PARTY}/3dmodels/1825910-6.STEP"
+		(model "${KIPRJMOD}/../Libraries/3dmodels/1825910-6.STEP"
 			(offset
 				(xyz 3.2 -2.2 0)
@@
 		)
 	)
-	(footprint "digikey-footprints:Switch_Tactile_THT_6x6mm_MJTP1230"
+	(footprint "RMP:Switch_Tactile_THT_6x6mm_MJTP1230"
 		(layer "F.Cu")
 		(at 78.925 99.9)
@@
 		)
 		(embedded_fonts no)
-		(model "${KICAD9_3RD_PARTY}/3dmodels/1825910-6.STEP"
+		(model "${KIPRJMOD}/../Libraries/3dmodels/1825910-6.STEP"
 			(offset
 				(xyz 3.2 -2.2 0)
@@
 		)
 	)
-	(footprint "Custom_Footprints:SOIC127P1032X265-24N"
+	(footprint "RMP:SOIC127P1032X265-24N"
 		(layer "B.Cu")
 		(at 82.72 65.785)
@@
 		)
 		(embedded_fonts no)
-		(model "${KICAD9_3RD_PARTY}/3dmodels/MAX7219CWGT.step"
+		(model "${KIPRJMOD}/../Libraries/3dmodels/MAX7219CWGT.step"
 			(offset
 				(xyz 0 0 0)
@@
 		)
 	)
-	(footprint "Custom_Footprints:SOIC127P1032X265-24N"
+	(footprint "RMP:SOIC127P1032X265-24N"
 		(layer "B.Cu")
 		(at 48.38 82.415)
@@
 		)
 		(embedded_fonts no)
-		(model "${KICAD9_3RD_PARTY}/3dmodels/MAX7219CWGT.step"
+		(model "${KIPRJMOD}/../Libraries/3dmodels/MAX7219CWGT.step"
 			(offset
 				(xyz 0 0 0)

Commit message: Chain the two MAX7219 on the MainPanel, as the built unit is wired
The schematic had both drivers on the MCU's DIN with a LOAD each (D67 for
the Active, D68 for the Standby) and both DOUT unconnected. The board in
use only works because two wires were added by hand: LOAD to LOAD, and
the Standby's DOUT to the Active's DIN. MobiFlight drives it as one LED
module of two devices on CS D68: connector 1 is the Standby, the first
in the chain, connector 2 the Active.

The design now matches:

  DIN         J9 pin 5 (D23) -> U2 (Standby) pin 1 only
  ACTIVE_DIN  U2 pin 24 (DOUT) -> U1 (Active) pin 1
  LOAD        J9 pin 6 (D68) -> U1 and U2 pin 12
  J9 pin 3    (D67) no longer used, flagged no-connect

The BoardPanel and the board config do not change. The old DIN branch
to U1 and the ACTIVE_LOAD track were removed; the two new connections
were routed interactively in KiCad (VHF2_BTN was shoved), then the GND
zones refilled. DRC: 0 unconnected, no clearance violation; the 15
remaining entries are the same library and field warnings as before.
Schematic parity unchanged.

On a board built from the old files, an Active display that shows the
odd wrong segment points at U1 pin 1: it is still tied to D23 by copper,
and with the hand wire it has two drivers.

Co-Authored-By: Claude Opus 5.5 <noreply@anthropic.com>
Connections:
- J9 pad 3: /Max7219 Displays/ACTIVE_LOAD -> unconnected-(J9-Pin_3-Pad3)
- J9 pad 6: /Max7219 Displays/STBY_LOAD -> /Max7219 Displays/LOAD
- U1 pad 1: /Max7219 Displays/DIN -> /Max7219 Displays/ACTIVE_DIN
- U1 pad 12: /Max7219 Displays/ACTIVE_LOAD -> /Max7219 Displays/LOAD
- U2 pad 12: /Max7219 Displays/STBY_LOAD -> /Max7219 Displays/LOAD
- U2 pad 24: unconnected-(U2-DOUT-Pad24) -> /Max7219 Displays/ACTIVE_DIN
Routing:
- net /Max7219 Displays/LOAD: track 0.00 -> 131.7 mm, vias 0 -> 3
- net /Max7219 Displays/ACTIVE_LOAD: track 103.5 -> 0.00 mm
- net /Max7219 Displays/STBY_LOAD: track 87.4 -> 0.00 mm, vias 2 -> 0
- net /Max7219 Displays/ACTIVE_DIN: track 0.00 -> 62.3 mm, vias 0 -> 6
- net /Max7219 Displays/DIN: track 114.5 -> 69.2 mm, vias 2 -> 0
- net /VHF2_BTN: track 81.9 -> 81.2 mm
