File: BoardPanel/BoardPanel.kicad_pcb (KiCad board)
At the start: 2 copper layers, 110 x 55 mm, 50 parts, among them J1 PJ-102A, J2 BootLoader, J3 Max 7219, J4 Led & Backlighting, J5 Main Button Board, J6 Cooling Fan, P1 USB_C_Plug_USB2.0, U1 ATMega2560, U2 P78A05-1000-THT, U3 CH340G

Commit message: Bring the custom parts into Libraries/, shared by all four boards
Six parts came from libraries that live only on the author's PC (SF
Library, IRLZ44N, P78A05-1000, Custom_Footprints, PCM_SFLibrary and the
Digi-Key PCM libraries). Their 3D models pointed at a KiCad 9 3rdparty
folder that no longer exists, so the boards rendered without them.

They now sit in Libraries/ under one nickname, RMP, as the overhead
panel does with OVHD:

  RMP.kicad_sym   MAX7219CWGT, IRLZ44NSTRLPBF, P78A05-1000, PJ-102A,
                  1825910-6, MJTP1230, taken from the schematic caches,
                  i.e. the symbols the boards were drawn with
  RMP.pretty      CONV_P78A05-1000, SOIC127P1032X265-24N,
                  TQFP100-0.5-14X14MM, NMOSGDS_D2PAK_INF, the PJ-102A
                  barrel jack and the MJTP1230 switch, copied from the
                  personal libraries (DRC found no difference from the
                  placed copies), with the 3D model of each board
                  instance added where the library had none
  3dmodels/       the seven vendor STEP files the boards use

Each board has a project sym-lib-table and fp-lib-table pointing at
${KIPRJMOD}/../Libraries, and every custom model path is now
${KIPRJMOD}/../Libraries/3dmodels/..., which resolves on any machine.

Netlists are unchanged apart from the library nickname in the footprint
field of U1, U2, S1, J1 (BoardPanel), Q1 (LedsPanel), U1, U2 and S1-S13
(MainPanel). Copper plots to the same geometry. ERC drops the missing-
library warnings: BoardPanel 4 -> 2, MainPanel 17 -> 2.

DRC no longer lists the malformed courtyard of the LedsPanel Q1, but its
courtyard still holds zero-length segments: it is fixed separately.

Co-Authored-By: Claude Opus 5.5 <noreply@anthropic.com>
Parts:
- J1: footprint digikey-footprints:Barrel_Jack_5.5mmODx2.1mmID_PJ-102A -> RMP:Barrel_Jack_5.5mmODx2.1mmID_PJ-102A
- S1: footprint digikey-footprints:Switch_Tactile_THT_6x6mm_MJTP1230 -> RMP:Switch_Tactile_THT_6x6mm_MJTP1230
- U1: footprint PCM_SFLibrary:TQFP100-0.5-14X14MM -> RMP:TQFP100-0.5-14X14MM
- U2: footprint Custom_Footprints:CONV_P78A05-1000 -> RMP:CONV_P78A05-1000
Changed lines of the file:
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@@
 		)
 	)
-	(footprint "digikey-footprints:Switch_Tactile_THT_6x6mm_MJTP1230"
+	(footprint "RMP:Switch_Tactile_THT_6x6mm_MJTP1230"
 		(layer "F.Cu")
 		(at 43.725 68.75)
@@
 		)
 		(embedded_fonts no)
-		(model "${KICAD9_3RD_PARTY}/3dmodels/1825910-6.STEP"
+		(model "${KIPRJMOD}/../Libraries/3dmodels/1825910-6.STEP"
 			(offset
 				(xyz 3.2 -2.2 0)
@@
 		)
 		(embedded_fonts no)
-		(model "${KICAD9_3RD_PARTY}/3dmodels/UJ2-BH-1-TH.STEP"
+		(model "${KIPRJMOD}/../Libraries/3dmodels/UJ2-BH-1-TH.STEP"
 			(offset
 				(xyz 14.5 -1 0.5)
@@
 		)
 	)
-	(footprint "Custom_Footprints:CONV_P78A05-1000"
+	(footprint "RMP:CONV_P78A05-1000"
 		(layer "F.Cu")
 		(at 102.1425 46.275)
@@
 		)
 		(embedded_fonts no)
-		(model "${KICAD9_3RD_PARTY}/3dmodels/P78A05-1000.step"
+		(model "${KIPRJMOD}/../Libraries/3dmodels/P78A05-1000.step"
 			(offset
 				(xyz 2.5 6.5 0.5)
@@
 		)
 	)
-	(footprint "digikey-footprints:Barrel_Jack_5.5mmODx2.1mmID_PJ-102A"
+	(footprint "RMP:Barrel_Jack_5.5mmODx2.1mmID_PJ-102A"
 		(layer "F.Cu")
 		(at 55.55 85.35 180)
@@
 		)
 		(embedded_fonts no)
-		(model "${KICAD9_3RD_PARTY}/3dmodels/PJ-102A.STEP"
+		(model "${KIPRJMOD}/../Libraries/3dmodels/PJ-102A.STEP"
 			(offset
 				(xyz 0 10.5 6.5)
@@
 		)
 	)
-	(footprint "PCM_SFLibrary:TQFP100-0.5-14X14MM"
+	(footprint "RMP:TQFP100-0.5-14X14MM"
 		(layer "F.Cu")
 		(at 64.875 55.05 45)
@@
 		)
 		(embedded_fonts no)
-		(model "${KICAD9_3RD_PARTY}/3dmodels/ATMEGA2560-16AU--3DModel-STEP-56544.STEP"
+		(model "${KIPRJMOD}/../Libraries/3dmodels/ATMEGA2560-16AU--3DModel-STEP-56544.STEP"
 			(offset
 				(xyz 0 0 0)

Commit message: Clear the ERC errors and the real DRC findings on all four boards
7Segments
- J5 used Conn_02x08_Top_Bottom_Shielded on an IDC header with no shield
  pad: ERC flagged the SH pin, DRC a net conflict. It is now the plain
  Conn_02x08_Top_Bottom, like J7/J8 on the MainPanel; pins 1-16 sit at
  the same points, so nothing else moved.
- GND had no driver: PWR_FLAG added.

BoardPanel
- P1 read "USB_C_Plug_USB2.0" on a USB-B connector: value now USB_B.
- +5V had no driver: pin 3 (+VOUT) of the P78A05 symbol is now a power
  output, in the schematic and in Libraries/RMP.kicad_sym. A PWR_FLAG
  there would clash with the pin.

MainPanel
- A stray no-connect flag and a second PWR_FLAG on the same net removed.

LedsPanel
- Q1 (IRLZ44N) pins were "unspecified": now passive, as in the overhead
  panel's library.
- Q1 courtyard: the two zero-length segments are gone, in the library
  footprint and on the board. The rest was already a closed outline
  around all three pads.
- J1 value on the board brought in line with the schematic (From_Main).

ERC is now 0 on 7Segments, LedsPanel and MainPanel. BoardPanel keeps one
warning, P1's USB_B symbol differing from the KiCad 10 library; that and
the DRC library/field mismatches go with Update Symbols/Footprints from
Library, as on the FCU. Netlists are unchanged apart from J5's SH node
and P1's value. Copper plots to the same geometry.

Co-Authored-By: Claude Opus 5.5 <noreply@anthropic.com>
Parts:
- P1: value USB_C_Plug_USB2.0 -> USB_B
Changed lines of the file:
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@@
 			)
 		)
-		(property "Value" "USB_C_Plug_USB2.0"
+		(property "Value" "USB_B"
 			(at 6.76 10.27 90)
 			(layer "F.Fab")
