File: BoardPanel/BoardPanel.kicad_sch (KiCad schematic)
At the start: 22 parts, among them J3 Max 7219, J4 Led & Backlighting, J5 Main Button Board, U1 ATMega2560

Commit message: Bring the custom parts into Libraries/, shared by all four boards
Six parts came from libraries that live only on the author's PC (SF
Library, IRLZ44N, P78A05-1000, Custom_Footprints, PCM_SFLibrary and the
Digi-Key PCM libraries). Their 3D models pointed at a KiCad 9 3rdparty
folder that no longer exists, so the boards rendered without them.

They now sit in Libraries/ under one nickname, RMP, as the overhead
panel does with OVHD:

  RMP.kicad_sym   MAX7219CWGT, IRLZ44NSTRLPBF, P78A05-1000, PJ-102A,
                  1825910-6, MJTP1230, taken from the schematic caches,
                  i.e. the symbols the boards were drawn with
  RMP.pretty      CONV_P78A05-1000, SOIC127P1032X265-24N,
                  TQFP100-0.5-14X14MM, NMOSGDS_D2PAK_INF, the PJ-102A
                  barrel jack and the MJTP1230 switch, copied from the
                  personal libraries (DRC found no difference from the
                  placed copies), with the 3D model of each board
                  instance added where the library had none
  3dmodels/       the seven vendor STEP files the boards use

Each board has a project sym-lib-table and fp-lib-table pointing at
${KIPRJMOD}/../Libraries, and every custom model path is now
${KIPRJMOD}/../Libraries/3dmodels/..., which resolves on any machine.

Netlists are unchanged apart from the library nickname in the footprint
field of U1, U2, S1, J1 (BoardPanel), Q1 (LedsPanel), U1, U2 and S1-S13
(MainPanel). Copper plots to the same geometry. ERC drops the missing-
library warnings: BoardPanel 4 -> 2, MainPanel 17 -> 2.

DRC no longer lists the malformed courtyard of the LedsPanel Q1, but its
courtyard still holds zero-length segments: it is fixed separately.

Co-Authored-By: Claude Opus 5.5 <noreply@anthropic.com>
Parts:
- S1: footprint digikey-footprints:Switch_Tactile_THT_6x6mm_MJTP1230 -> RMP:Switch_Tactile_THT_6x6mm_MJTP1230; symbol PCM_dk_Tactile-Switches:1825910-6 -> RMP:1825910-6
- U1: footprint PCM_SFLibrary:TQFP100-0.5-14X14MM -> RMP:TQFP100-0.5-14X14MM
Changed lines of the file:
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@@
 			)
 		)
-		(property "Footprint" "PCM_SFLibrary:TQFP100-0.5-14X14MM"
+		(property "Footprint" "RMP:TQFP100-0.5-14X14MM"
 			(at 128.27 95.25 0)
 			(hide yes)
@@
 	)
 	(symbol
-		(lib_id "PCM_dk_Tactile-Switches:1825910-6")
+		(lib_id "RMP:1825910-6")
 		(at 46.99 142.24 0)
 		(unit 1)
@@
 			)
 		)
-		(property "Footprint" "digikey-footprints:Switch_Tactile_THT_6x6mm_MJTP1230"
+		(property "Footprint" "RMP:Switch_Tactile_THT_6x6mm_MJTP1230"
 			(at 52.07 137.16 0)
 			(hide yes)
