File: BoardPanel/pwr_conn.kicad_sch (KiCad schematic)
At the start: 28 parts, among them J1 PJ-102A, J2 BootLoader, J6 Cooling Fan, P1 USB_C_Plug_USB2.0, U2 P78A05-1000-THT, U3 CH340G

Commit message: Bring the custom parts into Libraries/, shared by all four boards
Six parts came from libraries that live only on the author's PC (SF
Library, IRLZ44N, P78A05-1000, Custom_Footprints, PCM_SFLibrary and the
Digi-Key PCM libraries). Their 3D models pointed at a KiCad 9 3rdparty
folder that no longer exists, so the boards rendered without them.

They now sit in Libraries/ under one nickname, RMP, as the overhead
panel does with OVHD:

  RMP.kicad_sym   MAX7219CWGT, IRLZ44NSTRLPBF, P78A05-1000, PJ-102A,
                  1825910-6, MJTP1230, taken from the schematic caches,
                  i.e. the symbols the boards were drawn with
  RMP.pretty      CONV_P78A05-1000, SOIC127P1032X265-24N,
                  TQFP100-0.5-14X14MM, NMOSGDS_D2PAK_INF, the PJ-102A
                  barrel jack and the MJTP1230 switch, copied from the
                  personal libraries (DRC found no difference from the
                  placed copies), with the 3D model of each board
                  instance added where the library had none
  3dmodels/       the seven vendor STEP files the boards use

Each board has a project sym-lib-table and fp-lib-table pointing at
${KIPRJMOD}/../Libraries, and every custom model path is now
${KIPRJMOD}/../Libraries/3dmodels/..., which resolves on any machine.

Netlists are unchanged apart from the library nickname in the footprint
field of U1, U2, S1, J1 (BoardPanel), Q1 (LedsPanel), U1, U2 and S1-S13
(MainPanel). Copper plots to the same geometry. ERC drops the missing-
library warnings: BoardPanel 4 -> 2, MainPanel 17 -> 2.

DRC no longer lists the malformed courtyard of the LedsPanel Q1, but its
courtyard still holds zero-length segments: it is fixed separately.

Co-Authored-By: Claude Opus 5.5 <noreply@anthropic.com>
Parts:
- J1: footprint digikey-footprints:Barrel_Jack_5.5mmODx2.1mmID_PJ-102A -> RMP:Barrel_Jack_5.5mmODx2.1mmID_PJ-102A; symbol PCM_dk_Barrel-Power-Connectors:PJ-102A -> RMP:PJ-102A
- U2: footprint Custom_Footprints:CONV_P78A05-1000 -> RMP:CONV_P78A05-1000; symbol P78A05-1000:P78A05-1000 -> RMP:P78A05-1000
Changed lines of the file:
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@@
 	)
 	(symbol
-		(lib_id "PCM_dk_Barrel-Power-Connectors:PJ-102A")
+		(lib_id "RMP:PJ-102A")
 		(at 27.94 68.58 0)
 		(unit 1)
@@
 			)
 		)
-		(property "Footprint" "digikey-footprints:Barrel_Jack_5.5mmODx2.1mmID_PJ-102A"
+		(property "Footprint" "RMP:Barrel_Jack_5.5mmODx2.1mmID_PJ-102A"
 			(at 33.02 63.5 0)
 			(hide yes)
@@
 	)
 	(symbol
-		(lib_id "P78A05-1000:P78A05-1000")
+		(lib_id "RMP:P78A05-1000")
 		(at 95.25 168.91 0)
 		(unit 1)
@@
 			)
 		)
-		(property "Footprint" "Custom_Footprints:CONV_P78A05-1000"
+		(property "Footprint" "RMP:CONV_P78A05-1000"
 			(at 95.25 168.91 0)
 			(hide yes)

Commit message: Clear the ERC errors and the real DRC findings on all four boards
7Segments
- J5 used Conn_02x08_Top_Bottom_Shielded on an IDC header with no shield
  pad: ERC flagged the SH pin, DRC a net conflict. It is now the plain
  Conn_02x08_Top_Bottom, like J7/J8 on the MainPanel; pins 1-16 sit at
  the same points, so nothing else moved.
- GND had no driver: PWR_FLAG added.

BoardPanel
- P1 read "USB_C_Plug_USB2.0" on a USB-B connector: value now USB_B.
- +5V had no driver: pin 3 (+VOUT) of the P78A05 symbol is now a power
  output, in the schematic and in Libraries/RMP.kicad_sym. A PWR_FLAG
  there would clash with the pin.

MainPanel
- A stray no-connect flag and a second PWR_FLAG on the same net removed.

LedsPanel
- Q1 (IRLZ44N) pins were "unspecified": now passive, as in the overhead
  panel's library.
- Q1 courtyard: the two zero-length segments are gone, in the library
  footprint and on the board. The rest was already a closed outline
  around all three pads.
- J1 value on the board brought in line with the schematic (From_Main).

ERC is now 0 on 7Segments, LedsPanel and MainPanel. BoardPanel keeps one
warning, P1's USB_B symbol differing from the KiCad 10 library; that and
the DRC library/field mismatches go with Update Symbols/Footprints from
Library, as on the FCU. Netlists are unchanged apart from J5's SH node
and P1's value. Copper plots to the same geometry.

Co-Authored-By: Claude Opus 5.5 <noreply@anthropic.com>
Parts:
- P1: value USB_C_Plug_USB2.0 -> USB_B
Changed lines of the file:
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@@
 			)
 		)
-		(property "Value" "USB_C_Plug_USB2.0"
+		(property "Value" "USB_B"
 			(at 30.48 107.95 0)
 			(show_name no)

Commit message: Update symbols and footprints from the KiCad 10 libraries
Run in KiCad: Update Footprints from Library and Update PCB from
Schematic on all four boards, and Update Symbol from Library on P1 of
the BoardPanel only. Updating every symbol there would have reset the
ATmega's footprint field to the library default, as it did on the FCU.

  ERC      0 on all four boards
  DRC      0 on BoardPanel, LedsPanel and MainPanel; 15 silkscreen-
           clipped-by-mask warnings left on the 7Segments
  parity   0 everywhere; 0 unconnected

Every pad keeps its position and its net (IPC-D-356 compared before and
after on all 775 pads). Copper plots to the same coordinates. The only
netlist change is the one KiCad 10 makes to USB-B: P1's shield pin is
now 'SH' instead of '5', in the symbol and the footprint, still on GND.
The update also filled in the project name missing from three symbol
instances on the PowerConnectors sheet.

Update Footprints swapped P1's 3D model for the library's
USB_B_OST_USB-B1HSxx_Horizontal.step, which the KiCad 10 3D package does
not contain. The vendor UJ2-BH-1-TH model from Libraries/3dmodels is put
back, with its original offset and rotation.

Co-Authored-By: Claude Opus 5.5 <noreply@anthropic.com>
Connections:
- net GND: now also P1.SH (Shield); no longer P1.5 (Shield)
Changed lines of the file:
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@@
 		(pin "3"
 		)
-		(pin "5"
+		(pin "SH"
 		)
 		(pin "2"
@@
 		)
 		(instances
-			(project ""
+			(project "BoardPanel"
 				(path "/1f613cd0-8dd8-4e8e-b115-6705bccd9540/16b22287-4db5-4f68-a9f8-22977648d35e"
 					(reference "J6")
@@
 		)
 		(instances
-			(project ""
+			(project "BoardPanel"
 				(path "/1f613cd0-8dd8-4e8e-b115-6705bccd9540/16b22287-4db5-4f68-a9f8-22977648d35e"
 					(reference "#PWR05")
@@
 		)
 		(instances
-			(project ""
+			(project "BoardPanel"
 				(path "/1f613cd0-8dd8-4e8e-b115-6705bccd9540/16b22287-4db5-4f68-a9f8-22977648d35e"
 					(reference "U2")
